File: hardware/kicad/encoders.kicad_sch (KiCad schematic)
At the start: 8 parts, among them U3001 MCP23017x-x-SS, U3002 MCP23017x-x-SS

Commit message: WIP checkpoint commit before spliting the 5V rail
hardware/kicad/HALE-H8E10.kicad_pcb: Manufacturing: changed the board
  outline; tenting front back → -; covering - → -; plugging - → -;
  capping - → no; filling - → no; changed the plot output settings.
  Gergő Törcsvári: updated from the schematic (added C1003, C1004,
  C2001-C2016, C3001, C3002, C21001 and 83 more, TP1001-TP1003 not
  placed yet); placed C1003, C1004, C2001-C2016, C3001, C3002, C21001
  and 82 more; routed D_CS, DS_BL, DS_RES, E_INT and 86 more nets; added
  a zone on F.Cu, B.Cu; added a zone on F.Cu, B.Cu; added a zone on
  F.Cu, B.Cu; added a zone on F.Cu, B.Cu; and 15 more changes.
hardware/kicad/HALE-H8E10.kicad_pro: Manufacturing: max arc error - →
  0.005 mm; min connection width - → 0 mm; min groove width - → 0 mm;
  min microvia diameter - → 0.2 mm; min microvia drill - → 0.1 mm; min
  resolved spokes - → 2 mm; solder mask to copper clearance - → 0 mm;
  use height for length calcs - → true mm. Gergő Törcsvári: changed the
  predefined track widths (+4); changed the predefined diff pair sizes
  (+1); changed teardrop settings; changed default text and line
  settings; changed 62 DRC rule severities; changed DRC exclusions;
  changed schematic settings; changed 19 board.design settings settings.
hardware/kicad/HALE-H8E10.kicad_sch: Gergő Törcsvári added R1002, R1003
  and TP1001-TP1003 and wired them; removed C1001, C1002, C1005, D1001
  and D1002; changed C1004 value 100nF → 10uF; changed C1004 footprint
  Capacitor_SMD:C_0603_1608Metric_Pad1.08x0.95mm_HandSolder →
  Capacitor_SMD:C_0805_2012Metric_Pad1.18x1.45mm_HandSolder; changed
  C1004 LCSC C14663 → C15850; changed C1004 wiring (pins 1 and 2 now on
  GND and +5V); changed DS1001 wiring (pin 7 now on /D_CS); and 4 more
  changes.
hardware/kicad/encoders.kicad_sch: Gergő Törcsvári changed U3001 wiring;
  changed U3002 wiring; rearranged the sheet.
hardware/kicad/keys.kicad_sch: Gergő Törcsvári added TP2001 (3V3A) and
  wired it; change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
Connections:
- net ENC_A10: now also U3002.2 (GPB1); no longer U3002.6 (GPB5)
- net ENC_A6: now also U3001.6 (GPB5); no longer U3001.1 (GPB0)
- net ENC_A8: now also U3001.1 (GPB0); no longer U3001.6 (GPB5)
- net ENC_A9: now also U3002.5 (GPB4); no longer U3002.3 (GPB2)
- net ENC_B10: now also U3002.3 (GPB2); no longer U3002.7 (GPB6)
- net ENC_B6: now also U3001.7 (GPB6); no longer U3001.2 (GPB1)
- net ENC_B8: now also U3001.2 (GPB1); no longer U3001.7 (GPB6)
- net ENC_B9: now also U3002.6 (GPB5); no longer U3002.4 (GPB3)
- net ENC_SW10: now also U3002.1 (GPB0); no longer U3002.5 (GPB4)
- net ENC_SW8: now also U3002.7 (GPB6); no longer U3002.1 (GPB0)
- net ENC_SW9: now also U3002.4 (GPB3); no longer U3002.2 (GPB1)
Changed lines of the file:
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@@
 	)
 	(label "ENC_B6"
-		(at 86.36 74.93 0)
+		(at 86.36 87.63 0)
 		(effects
 			(font
@@
 	)
 	(label "ENC_A6"
-		(at 86.36 72.39 0)
+		(at 86.36 85.09 0)
 		(effects
 			(font
@@
 	)
 	(label "ENC_A8"
-		(at 86.36 85.09 0)
+		(at 86.36 72.39 0)
 		(effects
 			(font
@@
 	)
 	(label "ENC_SW8"
-		(at 88.9 156.21 0)
+		(at 87.63 171.45 0)
 		(effects
 			(font
@@
 	)
 	(label "ENC_B8"
-		(at 86.36 87.63 0)
+		(at 86.36 74.93 0)
 		(effects
 			(font
@@
 	)
 	(label "ENC_B9"
-		(at 88.9 163.83 0)
+		(at 87.63 168.91 0)
 		(effects
 			(font
@@
 	)
 	(label "ENC_SW9"
-		(at 88.9 158.75 0)
+		(at 87.63 163.83 0)
 		(effects
 			(font
@@
 	)
 	(label "ENC_A9"
-		(at 88.9 161.29 0)
+		(at 87.63 166.37 0)
 		(effects
 			(font
@@
 	)
 	(label "ENC_A10"
-		(at 88.9 168.91 0)
+		(at 87.63 158.75 0)
 		(effects
 			(font
@@
 	)
 	(label "ENC_B10"
-		(at 88.9 171.45 0)
+		(at 87.63 161.29 0)
 		(effects
 			(font
@@
 	)
 	(label "ENC_SW10"
-		(at 88.9 166.37 0)
+		(at 87.63 156.21 0)
 		(effects
 			(font
@@
 	(wire
 		(pts
-			(xy 80.01 72.39) (xy 86.36 72.39)
-		)
-		(stroke
-			(width 0)
-			(type default)
-		)
-	)
-	(wire
-		(pts
-			(xy 80.01 74.93) (xy 86.36 74.93)
-		)
-		(stroke
-			(width 0)
-			(type default)
-		)
-	)
-	(wire
-		(pts
 			(xy 80.01 77.47) (xy 86.36 77.47)
 		)
@@
 		(pts
 			(xy 80.01 82.55) (xy 86.36 82.55)
-		)
-		(stroke
-			(width 0)
-			(type default)
-		)
-	)
-	(wire
-		(pts
-			(xy 80.01 85.09) (xy 86.36 85.09)
-		)
-		(stroke
-			(width 0)
-			(type default)
-		)
-	)
-	(wire
-		(pts
-			(xy 80.01 87.63) (xy 86.36 87.63)
-		)
-		(stroke
-			(width 0)
-			(type default)
-		)
-	)
-	(wire
-		(pts
-			(xy 80.01 133.35) (xy 87.63 133.35)
-		)
-		(stroke
-			(width 0)
-			(type default)
-		)
-	)
-	(wire
-		(pts
-			(xy 80.01 135.89) (xy 87.63 135.89)
-		)
-		(stroke
-			(width 0)
-			(type default)
-		)
-	)
-	(wire
-		(pts
-			(xy 80.01 138.43) (xy 87.63 138.43)
-		)
-		(stroke
-			(width 0)
-			(type default)
-		)
-	)
-	(wire
-		(pts
-			(xy 80.01 140.97) (xy 87.63 140.97)
-		)
-		(stroke
-			(width 0)
-			(type default)
-		)
-	)
-	(wire
-		(pts
-			(xy 80.01 143.51) (xy 87.63 143.51)
-		)
-		(stroke
-			(width 0)
-			(type default)
-		)
-	)
-	(wire
-		(pts
-			(xy 80.01 146.05) (xy 87.63 146.05)
-		)
-		(stroke
-			(width 0)
-			(type default)
-		)
-	)
-	(wire
-		(pts
-			(xy 80.01 148.59) (xy 87.63 148.59)
-		)
-		(stroke
-			(width 0)
-			(type default)
-		)
-	)
-	(wire
-		(pts
-			(xy 80.01 156.21) (xy 88.9 156.21)
-		)
-		(stroke
-			(width 0)
-			(type default)
-		)
-	)
-	(wire
-		(pts
-			(xy 80.01 158.75) (xy 88.9 158.75)
-		)
-		(stroke
-			(width 0)
-			(type default)
-		)
-	)
-	(wire
-		(pts
-			(xy 80.01 161.29) (xy 88.9 161.29)
-		)
-		(stroke
-			(width 0)
-			(type default)
-		)
-	)
-	(wire
-		(pts
-			(xy 80.01 163.83) (xy 88.9 163.83)
-		)
-		(stroke
-			(width 0)
-			(type default)
-		)
-	)
-	(wire
-		(pts
-			(xy 80.01 166.37) (xy 88.9 166.37)
-		)
-		(stroke
-			(width 0)
-			(type default)
-		)
-	)
-	(wire
-		(pts
-			(xy 80.01 168.91) (xy 88.9 168.91)
-		)
-		(stroke
-			(width 0)
-			(type default)
-		)
-	)
-	(wire
-		(pts
-			(xy 80.01 171.45) (xy 88.9 171.45)
 		)
 		(stroke
@@
 		)
 		(stroke
+			(width 0)
+			(type default)
+		)
+	)
+	(wire
+		(pts
+			(xy 80.01 171.45) (xy 87.63 171.45)
+		)
+		(stroke
+			(width 0)
+			(type default)
+		)
+	)
+	(wire
+		(pts
+			(xy 80.01 168.91) (xy 87.63 168.91)
+		)
+		(stroke
+			(width 0)
+			(type default)
+		)
+	)
+	(wire
+		(pts
+			(xy 80.01 166.37) (xy 87.63 166.37)
+		)
+		(stroke
+			(width 0)
+			(type default)
+		)
+	)
+	(wire
+		(pts
+			(xy 80.01 163.83) (xy 87.63 163.83)
+		)
+		(stroke
+			(width 0)
+			(type default)
+		)
+	)
+	(wire
+		(pts
+			(xy 80.01 161.29) (xy 87.63 161.29)
+		)
+		(stroke
+			(width 0)
+			(type default)
+		)
+	)
+	(wire
+		(pts
+			(xy 80.01 158.75) (xy 87.63 158.75)
+		)
+		(stroke
+			(width 0)
+			(type default)
+		)
+	)
+	(wire
+		(pts
+			(xy 80.01 156.21) (xy 87.63 156.21)
+		)
+		(stroke
+			(width 0)
+			(type default)
+		)
+	)
+	(wire
+		(pts
+			(xy 80.01 148.59) (xy 87.63 148.59)
+		)
+		(stroke
+			(width 0)
+			(type default)
+		)
+	)
+	(wire
+		(pts
+			(xy 80.01 146.05) (xy 87.63 146.05)
+		)
+		(stroke
+			(width 0)
+			(type default)
+		)
+	)
+	(wire
+		(pts
+			(xy 80.01 143.51) (xy 87.63 143.51)
+		)
+		(stroke
+			(width 0)
+			(type default)
+		)
+	)
+	(wire
+		(pts
+			(xy 80.01 140.97) (xy 87.63 140.97)
+		)
+		(stroke
+			(width 0)
+			(type default)
+		)
+	)
+	(wire
+		(pts
+			(xy 80.01 138.43) (xy 87.63 138.43)
+		)
+		(stroke
+			(width 0)
+			(type default)
+		)
+	)
+	(wire
+		(pts
+			(xy 80.01 135.89) (xy 87.63 135.89)
+		)
+		(stroke
+			(width 0)
+			(type default)
+		)
+	)
+	(wire
+		(pts
+			(xy 80.01 133.35) (xy 87.63 133.35)
+		)
+		(stroke
+			(width 0)
+			(type default)
+		)
+	)
+	(wire
+		(pts
+			(xy 80.01 72.39) (xy 86.36 72.39)
+		)
+		(stroke
+			(width 0)
+			(type default)
+		)
+	)
+	(wire
+		(pts
+			(xy 80.01 74.93) (xy 86.36 74.93)
+		)
+		(stroke
+			(width 0)
+			(type default)
+		)
+	)
+	(wire
+		(pts
+			(xy 80.01 85.09) (xy 86.36 85.09)
+		)
+		(stroke
+			(width 0)
+			(type default)
+		)
+	)
+	(wire
+		(pts
+			(xy 80.01 87.63) (xy 86.36 87.63)
+		)
+		(stroke

Commit message: "finished" PCB
hardware/kicad/HALE-H8E10.kicad_pcb: Manufacturing: changed the board
  outline. Gergő Törcsvári: updated from the schematic (added C1001,
  C1002, C1004-C1009, H1001-H1012, R1004, R1005 and 5 more; removed
  R1002 and R1003; nets changed on 44 pads); placed C1001, C1002,
  C1004-C1009, H1001-H1012, R1004, R1005 and 4 more; added REF**;
  removed C1004; moved C1003, C2002, C2003, C2006, R1001, TP2001 and
  U1001; routed EN_AUX, EN_LED, +5V_AUX, +5V_LED and 3 more nets;
  rerouted D_CS, DS_BL, DS_RES, E_INT and 21 more nets; and 3 more
  changes.
hardware/kicad/HALE-H8E10.kicad_pro: Gergő Törcsvári excluded 2 DRC
  violations; changed schematic settings.
hardware/kicad/HALE-H8E10.kicad_sch: Gergő Törcsvári added C1001, C1002,
  C1005-C1009, H1001-H1012, R1004, R1005 and 4 more and wired them;
  removed R1002 and R1003; changed 4 parts' fields; changed C1004 wiring
  (pin 1 now on +5V); renamed net unconnected-(U1002-D3-Pad4) to
  /EN_AUX; renamed net unconnected-(U1002-D15-Pad19) to /EN_LED; split
  +5V into +5V_AUX and +5V_LED; and 4 more changes.
hardware/kicad/encoder.kicad_sch: Gergő Törcsvári changed 10 parts'
  fields; renamed net unconnected-(U1002-D3-Pad4) to /EN_AUX; renamed
  net unconnected-(U1002-D15-Pad19) to /EN_LED; split +5V into +5V_AUX
  and +5V_LED.
hardware/kicad/encoders.kicad_sch: Gergő Törcsvári changed 6 parts'
  fields; renamed net unconnected-(U1002-D3-Pad4) to /EN_AUX; renamed
  net unconnected-(U1002-D15-Pad19) to /EN_LED; split +5V into +5V_AUX
  and +5V_LED.
hardware/kicad/key_cell.kicad_sch: Gergő Törcsvári changed 16 parts'
  fields; renamed net unconnected-(U1002-D3-Pad4) to /EN_AUX; renamed
  net unconnected-(U1002-D15-Pad19) to /EN_LED; split +5V into +5V_AUX
  and +5V_LED.
hardware/kicad/keys.kicad_sch: Gergő Törcsvári added R2001 (10K) and
  wired it to /KEYS_CS; changed 6 parts' fields; renamed net
  unconnected-(U1002-D3-Pad4) to /EN_AUX; renamed net
  unconnected-(U1002-D15-Pad19) to /EN_LED; split +5V into +5V_A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
Parts:
- R3001, R3002: LCSC (none) -> C23162
- R3003, R3004: LCSC (none) -> C25804
- U3001, U3002: LCSC (none) -> C506653
Changed lines of the file:
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@@
 			)
 		)
-		(property "LCSC" ""
+		(property "LCSC" "C506653"
 			(at 67.31 69.85 0)
 			(hide yes)
@@
 			)
 		)
-		(property "LCSC" ""
+		(property "LCSC" "C506653"
 			(at 67.31 153.67 0)
 			(hide yes)
@@
 			)
 		)
-		(property "LCSC" ""
+		(property "LCSC" "C25804"
 			(at 34.29 72.39 90)
 			(hide yes)
@@
 			)
 		)
-		(property "LCSC" ""
+		(property "LCSC" "C25804"
 			(at 33.02 59.69 90)
 			(hide yes)
@@
 			)
 		)
-		(property "LCSC" ""
+		(property "LCSC" "C23162"
 			(at 24.13 34.29 90)
 			(hide yes)
@@
 			)
 		)
-		(property "LCSC" ""
+		(property "LCSC" "C23162"
 			(at 24.13 25.4 90)
 			(hide yes)
