File: hardware/kicad/HALE-H8E10.kicad_pcb (KiCad board)
At the start: 2 copper layers, 217 x 77.7 mm, 157 parts, among them K21001 ks-20, K22001 ks-20, K23001 ks-20, K24001 ks-20, K25001 ks-20, K26001 ks-20, K27001 ks-20, K28001 ks-20, SW31001 RotaryEncoder_Switch_MP, SW32001 RotaryEncoder_Switch_MP, SW33001 RotaryEncoder_Switch_MP, SW34001 RotaryEncoder_Switch_MP, SW35001 RotaryEncoder_Switch_MP, SW36001 RotaryEncoder_Switch_MP, SW37001 RotaryEncoder_Switch_MP, SW38001 RotaryEncoder_Switch_MP, SW39001 RotaryEncoder_Switch_MP, SW40001 RotaryEncoder_Switch_MP, U1001 74AHCT1G125, U1002 XIAO-ESP32-S3-Plus-SMD, U1003 TPS22810DBV, U1004 TPS22810DBV, U2001 ME6211C33M5, U2002 MCP3208, U21001 DRV5055A3xDBZxQ1, U22001 DRV5055A3xDBZxQ1, U23001 DRV5055A3xDBZxQ1, U24001 DRV5055A3xDBZxQ1, U25001 DRV5055A3xDBZxQ1, U26001 DRV5055A3xDBZxQ1, U27001 DRV5055A3xDBZxQ1, U28001 DRV5055A3xDBZxQ1, U3001 MCP23017x-x-SS, U3002 MCP23017x-x-SS

Commit message: rev, and minor adjustements
hardware/kicad/HALE-H8E10.kicad_pcb: Gergő Törcsvári moved K21001,
  K22001, K23001, K24001, K25001, K26001, K27001 and K28001; title
  block: date - → ${RELEASE_DATE}, rev - → ${REV}, title - → HALE-H8E10;
  tidied the silkscreen.
hardware/kicad/HALE-H8E10.kicad_pro: Manufacturing: changed the IPC-2581
  settings. Gergő Törcsvári: RELEASE_DATE - → 2026-10-20; REV - → 1.0;
  changed schematic settings.
hardware/kicad/HALE-H8E10.kicad_sch: Gergő Törcsvári title block: date
  2026-10-12 → ${RELEASE_DATE}, rev A → ${REV}.
hardware/kicad/encoder.kicad_sch: Gergő Törcsvári changed 10 parts'
  fields.
hardware/kicad/key_cell.kicad_sch: Gergő Törcsvári changed 8 parts'
  fields.
hardware/kicad/pcbjam.lock.json: Library lockfile regenerated.

Checks: ERC: 2 errors in HALE-H8E10.kicad_sch (pin to pin ×2) · DRC clean

PCBJam-Commit: 7f3340a3-7d55-4157-ad73-e17d7d28c5bf
Parts:
- renumbered REF** to LogoB, REF** to LogoF
Other:
- board text added: "Rev ${REV} - ${RELEASE_DATE}"
- board text removed: "Rev 1.0 - 2026.10.19."
Changed lines of the file:
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@@
 	(property "FAB" "JLCPCB")
 	(property "FAB_PROFILE" "jlcpcb v3 (standard)")
+	(property "RELEASE_DATE" "2026-10-20")
+	(property "REV" "1.0")
 	(embedded_fonts no)
+	(title_block
+		(title "HALE-H8E10")
+		(date "${RELEASE_DATE}")
+		(rev "${REV}")
+	)
 	(gr_rect
 		(start 26.5 61.16)
@@
 			)
 		)
-		(property "LCSC" "C5378731"
+		(property "LCSC" "C5149201"
 			(at 0 0 0)
 			(unlocked yes)
@@
 		(locked yes)
 		(layer "F.Cu")
-		(at 98.075 125.315)
+		(at 98.1 125.315)
 		(property "Reference" "K28001"
 			(at 0 -0.5 0)
@@
 		(locked yes)
 		(layer "F.Cu")
-		(at 40.925 106.265)
+		(at 40.95 106.265)
 		(property "Reference" "K21001"
 			(at 0 -0.5 0)
@@
 			)
 		)
-		(property "LCSC" "C5378731"
+		(property "LCSC" "C5149201"
 			(at 0 0 180)
 			(unlocked yes)
@@
 			)
 		)
-		(property "LCSC" "C5378731"
+		(property "LCSC" "C5149201"
 			(at 0 0 180)
 			(unlocked yes)
@@
 		(locked yes)
 		(layer "F.Cu")
-		(at 79.025 106.265)
+		(at 79.05 106.265)
 		(property "Reference" "K23001"
 			(at 0 -0.5 0)
@@
 		(locked yes)
 		(layer "F.Cu")
-		(at 59.975 125.315)
+		(at 60 125.315)
 		(property "Reference" "K26001"
 			(at 0 -0.5 0)
@@
 			)
 		)
-		(property "LCSC" "C5378731"
+		(property "LCSC" "C5149201"
 			(at 0 0 180)
 			(unlocked yes)
@@
 		(locked yes)
 		(layer "F.Cu")
-		(at 40.925 125.315)
+		(at 40.95 125.315)
 		(property "Reference" "K25001"
 			(at 0 -0.5 0)
@@
 			)
 		)
-		(property "LCSC" "C5378731"
+		(property "LCSC" "C5149201"
 			(at 0 0 180)
 			(unlocked yes)
@@
 			)
 		)
-		(property "LCSC" "C5378731"
+		(property "LCSC" "C5149201"
 			(at 0 0 180)
 			(unlocked yes)
@@
 		(sheetname "/")
 		(sheetfile "HALE-H8E10.kicad_sch")
+		(units
+			(unit
+				(name "A")
+				(pins "1" "2" "3" "4" "5" "6" "7" "15" "16" "17" "18" "24" "25" "26"
+					"32" "27" "33" "28" "34" "29" "30" "31" "14" "13" "12" "11" "10" "9"
+					"8" "23" "22" "21" "20" "19"
+				)
+			)
+		)
 		(attr smd)
 		(duplicate_pad_numbers_are_jumpers no)
@@
 			(at 0 1.43 0)
 			(layer "B.SilkS")
+			(hide yes)
 			(effects
 				(font
@@
 			)
 		)
-		(property "LCSC" "C5378731"
+		(property "LCSC" "C5149201"
 			(at 0 0 0)
 			(unlocked yes)
@@
 			)
 		)
-		(property "LCSC" "C5378731"
+		(property "LCSC" "C5149201"
 			(at 0 0 0)
 			(unlocked yes)
@@
 			)
 		)
-		(property "LCSC" "C5378731"
+		(property "LCSC" "C5149201"
 			(at 0 0 0)
 			(unlocked yes)
@@
 		(locked yes)
 		(layer "F.Cu")
-		(at 98.075 106.265)
+		(at 98.1 106.265)
 		(property "Reference" "K24001"
 			(at 0 -0.5 0)
@@
 			)
 		)
-		(property "LCSC" "C5378731"
+		(property "LCSC" "C5149201"
 			(at 0 0 180)
 			(unlocked yes)
@@
 			)
 		)
-		(property "LCSC" "C5378731"
+		(property "LCSC" "C5149201"
 			(at 0 0 180)
 			(unlocked yes)
@@
 			)
 		)
-		(property "LCSC" "C5378731"
+		(property "LCSC" "C5149201"
 			(at 0 0 180)
 			(unlocked yes)
@@
 		(locked yes)
 		(layer "F.Cu")
-		(at 79.025 125.315)
+		(at 79.05 125.315)
 		(property "Reference" "K27001"
 			(at 0 -0.5 0)
@@
 			)
 		)
-		(property "LCSC" "C5378731"
+		(property "LCSC" "C5149201"
 			(at 0 0 180)
 			(unlocked yes)
@@
 			)
 		)
-		(property "LCSC" "C5378731"
+		(property "LCSC" "C5149201"
 			(at 0 0 180)
 			(unlocked yes)
@@
 			)
 		)
-		(property "LCSC" "C5378731"
+		(property "LCSC" "C5149201"
 			(at 0 0 180)
 			(unlocked yes)
@@
 			)
 		)
-		(property "LCSC" "C5378731"
+		(property "LCSC" "C5149201"
 			(at 0 0 0)
 			(unlocked yes)
@@
 			)
 		)
-		(property "LCSC" "C5378731"
+		(property "LCSC" "C5149201"
 			(at 0 0 180)
 			(unlocked yes)
@@
 		(locked yes)
 		(layer "F.Cu")
-		(at 59.975 106.265)
+		(at 60 106.265)
 		(property "Reference" "K22001"
 			(at 0 -0.5 0)
@@
 			)
 		)
-		(property "LCSC" "C5378731"
+		(property "LCSC" "C5149201"
 			(at 0 0 180)
 			(unlocked yes)
@@
 		(layer "B.Cu")
 		(at 69.5 93.458 180)
-		(property "Reference" "REF**"
+		(property "Reference" "LogoB"
 			(at 0 0.5 0)
 			(unlocked yes)
@@
 			)
 		)
-		(attr through_hole)
 		(duplicate_pad_numbers_are_jumpers no)
 		(fp_line
@@
 		(layer "F.Cu")
 		(at 70.5 93.5)
-		(property "Reference" "REF**"
+		(property "Reference" "LogoF"
 			(at 0 -0.5 0)
 			(unlocked yes)
@@
 			)
 		)
-		(attr through_hole)
 		(duplicate_pad_numbers_are_jumpers no)
 		(fp_line
@@
 		(embedded_fonts no)
 	)
-	(gr_text "Rev 1.0 - 2026.10.19."
-		(at 62.5 135.5 0)
+	(gr_text "Rev ${REV} - ${RELEASE_DATE}"
+		(at 63.5 135.5 0)
 		(layer "B.SilkS")
 		(effects
