File: hardware/kicad/key_cell.kicad_sch (KiCad schematic)
At the start: 5 parts, among them K21001 ks-20, U21001 DRV5055A3xDBZxQ1

Commit message: "finished" PCB
hardware/kicad/HALE-H8E10.kicad_pcb: Manufacturing: changed the board
  outline. Gergő Törcsvári: updated from the schematic (added C1001,
  C1002, C1004-C1009, H1001-H1012, R1004, R1005 and 5 more; removed
  R1002 and R1003; nets changed on 44 pads); placed C1001, C1002,
  C1004-C1009, H1001-H1012, R1004, R1005 and 4 more; added REF**;
  removed C1004; moved C1003, C2002, C2003, C2006, R1001, TP2001 and
  U1001; routed EN_AUX, EN_LED, +5V_AUX, +5V_LED and 3 more nets;
  rerouted D_CS, DS_BL, DS_RES, E_INT and 21 more nets; and 3 more
  changes.
hardware/kicad/HALE-H8E10.kicad_pro: Gergő Törcsvári excluded 2 DRC
  violations; changed schematic settings.
hardware/kicad/HALE-H8E10.kicad_sch: Gergő Törcsvári added C1001, C1002,
  C1005-C1009, H1001-H1012, R1004, R1005 and 4 more and wired them;
  removed R1002 and R1003; changed 4 parts' fields; changed C1004 wiring
  (pin 1 now on +5V); renamed net unconnected-(U1002-D3-Pad4) to
  /EN_AUX; renamed net unconnected-(U1002-D15-Pad19) to /EN_LED; split
  +5V into +5V_AUX and +5V_LED; and 4 more changes.
hardware/kicad/encoder.kicad_sch: Gergő Törcsvári changed 10 parts'
  fields; renamed net unconnected-(U1002-D3-Pad4) to /EN_AUX; renamed
  net unconnected-(U1002-D15-Pad19) to /EN_LED; split +5V into +5V_AUX
  and +5V_LED.
hardware/kicad/encoders.kicad_sch: Gergő Törcsvári changed 6 parts'
  fields; renamed net unconnected-(U1002-D3-Pad4) to /EN_AUX; renamed
  net unconnected-(U1002-D15-Pad19) to /EN_LED; split +5V into +5V_AUX
  and +5V_LED.
hardware/kicad/key_cell.kicad_sch: Gergő Törcsvári changed 16 parts'
  fields; renamed net unconnected-(U1002-D3-Pad4) to /EN_AUX; renamed
  net unconnected-(U1002-D15-Pad19) to /EN_LED; split +5V into +5V_AUX
  and +5V_LED.
hardware/kicad/keys.kicad_sch: Gergő Törcsvári added R2001 (10K) and
  wired it to /KEYS_CS; changed 6 parts' fields; renamed net
  unconnected-(U1002-D3-Pad4) to /EN_AUX; renamed net
  unconnected-(U1002-D15-Pad19) to /EN_LED; split +5V into +5V_A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
Parts:
- D21001: LCSC (none) -> C5378731
- U21001: LCSC (none) -> C266128
Connections:
- net +5V renamed +5V_LED
Changed lines of the file:
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@@
 			)
 		)
-		(property "LCSC" ""
+		(property "LCSC" "C266128"
 			(at 93.98 102.87 0)
 			(hide yes)
@@
 			)
 		)
-		(property "LCSC" ""
+		(property "LCSC" "C5378731"
 			(at 144.78 102.87 0)
 			(hide yes)
@@
 	)
 	(symbol
-		(lib_id "power:+5V")
-		(at 144.78 80.01 0)
-		(unit 1)
-		(body_style 1)
-		(exclude_from_sim no)
-		(in_bom yes)
-		(on_board yes)
-		(in_pos_files yes)
-		(dnp no)
-		(fields_autoplaced yes)
-		(property "Reference" "#PWR021004"
-			(at 144.78 83.82 0)
-			(hide yes)
-			(show_name no)
-			(do_not_autoplace no)
-			(effects
-				(font
-					(size 1.27 1.27)
-				)
-			)
-		)
-		(property "Value" "+5V"
-			(at 144.78 74.93 0)
-			(show_name no)
-			(do_not_autoplace no)
-			(effects
-				(font
-					(size 1.27 1.27)
-				)
-			)
-		)
-		(property "Footprint" ""
-			(at 144.78 80.01 0)
-			(hide yes)
-			(show_name no)
-			(do_not_autoplace no)
-			(effects
-				(font
-					(size 1.27 1.27)
-				)
-			)
-		)
-		(property "Datasheet" ""
-			(at 144.78 80.01 0)
-			(hide yes)
-			(show_name no)
-			(do_not_autoplace no)
-			(effects
-				(font
-					(size 1.27 1.27)
-				)
-			)
-		)
-		(property "Description" "Power symbol creates a global label with name \"+5V\""
-			(at 144.78 80.01 0)
-			(hide yes)
-			(show_name no)
-			(do_not_autoplace no)
-			(effects
-				(font
-					(size 1.27 1.27)
-				)
-			)
-		)
-		(pin "1"
-		)
-		(instances
-			(project "HALE-H8E10"
-				(path "/95d89127-9479-4179-8532-6fc4e4c352d8/4b75bd9e-329e-4489-b23d-ebc8bc921298/1f925e4c-dce3-4ac5-9354-f83a74aac100"
-					(reference "#PWR028004")
-					(unit 1)
-				)
-				(path "/95d89127-9479-4179-8532-6fc4e4c352d8/4b75bd9e-329e-4489-b23d-ebc8bc921298/2dc657e5-15fd-41e0-b47b-75b61abb9356"
-					(reference "#PWR024004")
-					(unit 1)
-				)
-				(path "/95d89127-9479-4179-8532-6fc4e4c352d8/4b75bd9e-329e-4489-b23d-ebc8bc921298/6bd8124a-9a6a-49a7-a7f6-e58e6c394933"
-					(reference "#PWR023004")
-					(unit 1)
-				)
-				(path "/95d89127-9479-4179-8532-6fc4e4c352d8/4b75bd9e-329e-4489-b23d-ebc8bc921298/8706e16d-fdf1-444d-8a94-f5654ae49972"
-					(reference "#PWR021004")
-					(unit 1)
-				)
-				(path "/95d89127-9479-4179-8532-6fc4e4c352d8/4b75bd9e-329e-4489-b23d-ebc8bc921298/888e8f29-2925-45e8-a00f-bfff82b2556a"
-					(reference "#PWR027004")
-					(unit 1)
-				)
-				(path "/95d89127-9479-4179-8532-6fc4e4c352d8/4b75bd9e-329e-4489-b23d-ebc8bc921298/89893055-74b7-4945-8ab7-222602d7eedd"
-					(reference "#PWR026004")
-					(unit 1)
-				)
-				(path "/95d89127-9479-4179-8532-6fc4e4c352d8/4b75bd9e-329e-4489-b23d-ebc8bc921298/c9f921a4-2ce9-4a28-887f-fad0b6a1581c"
-					(reference "#PWR022004")
-					(unit 1)
-				)
-				(path "/95d89127-9479-4179-8532-6fc4e4c352d8/4b75bd9e-329e-4489-b23d-ebc8bc921298/fc6ddc38-42a7-4ac8-a817-625672ab43c2"
-					(reference "#PWR025004")
-					(unit 1)
-				)
-			)
-		)
-	)
-	(symbol
 		(lib_id "power:GND")
 		(at 144.78 115.57 0)
@@
 		)
 	)
+	(symbol
+		(lib_id "power:+5VL")
+		(at 144.78 80.01 0)
+		(unit 1)
+		(body_style 1)
+		(exclude_from_sim no)
+		(in_bom yes)
+		(on_board yes)
+		(in_pos_files yes)
+		(dnp no)
+		(fields_autoplaced yes)
+		(property "Reference" "#PWR021004"
+			(at 144.78 83.82 0)
+			(hide yes)
+			(show_name no)
+			(do_not_autoplace no)
+			(effects
+				(font
+					(size 1.27 1.27)
+				)
+			)
+		)
+		(property "Value" "+5V_LED"
+			(at 144.78 74.93 0)
+			(show_name no)
+			(do_not_autoplace no)
+			(effects
+				(font
+					(size 1.27 1.27)
+				)
+			)
+		)
+		(property "Footprint" ""
+			(at 144.78 80.01 0)
+			(hide yes)
+			(show_name no)
+			(do_not_autoplace no)
+			(effects
+				(font
+					(size 1.27 1.27)
+				)
+			)
+		)
+		(property "Datasheet" ""
+			(at 144.78 80.01 0)
+			(hide yes)
+			(show_name no)
+			(do_not_autoplace no)
+			(effects
+				(font
+					(size 1.27 1.27)
+				)
+			)
+		)
+		(property "Description" "Power symbol creates a global label with name \"+5VL\""
+			(at 144.78 80.01 0)
+			(hide yes)
+			(show_name no)
+			(do_not_autoplace no)
+			(effects
+				(font
+					(size 1.27 1.27)
+				)
+			)
+		)
+		(pin "1"
+		)
+		(instances
+			(project "HALE-H8E10"
+				(path "/95d89127-9479-4179-8532-6fc4e4c352d8/4b75bd9e-329e-4489-b23d-ebc8bc921298/1f925e4c-dce3-4ac5-9354-f83a74aac100"
+					(reference "#PWR028004")
+					(unit 1)
+				)
+				(path "/95d89127-9479-4179-8532-6fc4e4c352d8/4b75bd9e-329e-4489-b23d-ebc8bc921298/2dc657e5-15fd-41e0-b47b-75b61abb9356"
+					(reference "#PWR024004")
+					(unit 1)
+				)
+				(path "/95d89127-9479-4179-8532-6fc4e4c352d8/4b75bd9e-329e-4489-b23d-ebc8bc921298/6bd8124a-9a6a-49a7-a7f6-e58e6c394933"
+					(reference "#PWR023004")
+					(unit 1)
+				)
+				(path "/95d89127-9479-4179-8532-6fc4e4c352d8/4b75bd9e-329e-4489-b23d-ebc8bc921298/8706e16d-fdf1-444d-8a94-f5654ae49972"
+					(reference "#PWR021004")
+					(unit 1)
+				)
+				(path "/95d89127-9479-4179-8532-6fc4e4c352d8/4b75bd9e-329e-4489-b23d-ebc8bc921298/888e8f29-2925-45e8-a00f-bfff82b2556a"
+					(reference "#PWR027004")
+					(unit 1)
+				)
+				(path "/95d89127-9479-4179-8532-6fc4e4c352d8/4b75bd9e-329e-4489-b23d-ebc8bc921298/89893055-74b7-4945-8ab7-222602d7eedd"
+					(reference "#PWR026004")
+					(unit 1)
+				)
+				(path "/95d89127-9479-4179-8532-6fc4e4c352d8/4b75bd9e-329e-4489-b23d-ebc8bc921298/c9f921a4-2ce9-4a28-887f-fad0b6a1581c"
+					(reference "#PWR022004")
+					(unit 1)
+				)
+				(path "/95d89127-9479-4179-8532-6fc4e4c352d8/4b75bd9e-329e-4489-b23d-ebc8bc921298/fc6ddc38-42a7-4ac8-a817-625672ab43c2"
+					(reference "#PWR025004")
+					(unit 1)
+				)
+			)
+		)
+	)

Commit message: rev, and minor adjustements
hardware/kicad/HALE-H8E10.kicad_pcb: Gergő Törcsvári moved K21001,
  K22001, K23001, K24001, K25001, K26001, K27001 and K28001; title
  block: date - → ${RELEASE_DATE}, rev - → ${REV}, title - → HALE-H8E10;
  tidied the silkscreen.
hardware/kicad/HALE-H8E10.kicad_pro: Manufacturing: changed the IPC-2581
  settings. Gergő Törcsvári: RELEASE_DATE - → 2026-10-20; REV - → 1.0;
  changed schematic settings.
hardware/kicad/HALE-H8E10.kicad_sch: Gergő Törcsvári title block: date
  2026-10-12 → ${RELEASE_DATE}, rev A → ${REV}.
hardware/kicad/encoder.kicad_sch: Gergő Törcsvári changed 10 parts'
  fields.
hardware/kicad/key_cell.kicad_sch: Gergő Törcsvári changed 8 parts'
  fields.
hardware/kicad/pcbjam.lock.json: Library lockfile regenerated.

Checks: ERC: 2 errors in HALE-H8E10.kicad_sch (pin to pin ×2) · DRC clean

PCBJam-Commit: 7f3340a3-7d55-4157-ad73-e17d7d28c5bf
Parts:
- D21001: LCSC C5378731 -> C5149201
Changed lines of the file:
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@@
 			)
 		)
-		(property "LCSC" "C5378731"
+		(property "LCSC" "C5149201"
 			(at 144.78 102.87 0)
 			(hide yes)
