File: hardware/H4E2/H4E2.kicad_pcb (KiCad board)
At the start: 2 copper layers, 217 x 77.7 mm, 157 parts, among them K21001 ks-20, K22001 ks-20, K23001 ks-20, K24001 ks-20, K25001 ks-20, K26001 ks-20, K27001 ks-20, K28001 ks-20, SW31001 RotaryEncoder_Switch_MP, SW32001 RotaryEncoder_Switch_MP, SW33001 RotaryEncoder_Switch_MP, SW34001 RotaryEncoder_Switch_MP, SW35001 RotaryEncoder_Switch_MP, SW36001 RotaryEncoder_Switch_MP, SW37001 RotaryEncoder_Switch_MP, SW38001 RotaryEncoder_Switch_MP, SW39001 RotaryEncoder_Switch_MP, SW40001 RotaryEncoder_Switch_MP, U1001 74AHCT1G125, U1002 XIAO-ESP32-S3-Plus-SMD, U1003 TPS22810DBV, U1004 TPS22810DBV, U2001 ME6211C33M5, U2002 MCP3208, U21001 DRV5055A3xDBZxQ1, U22001 DRV5055A3xDBZxQ1, U23001 DRV5055A3xDBZxQ1, U24001 DRV5055A3xDBZxQ1, U25001 DRV5055A3xDBZxQ1, U26001 DRV5055A3xDBZxQ1, U27001 DRV5055A3xDBZxQ1, U28001 DRV5055A3xDBZxQ1, U3001 MCP23017x-x-SS, U3002 MCP23017x-x-SS

Commit message: H4E2 "final" design.
hardware/H4E2/H4E2.kicad_pcb: Manufacturing: changed the board outline.
  Gergő Törcsvári: updated from the schematic (added C1008, C1009,
  H1005, R2002-R2005, TP1001, TP1003 and TP1004; removed C2004, C2008,
  C2010, C2013, C3002, C23001 and 47 more; nets changed on 28 pads);
  placed C1008, C1009, C3001, C31001-C31003, C36001-C36003, D31001 and
  10 more; added REF**; removed C1008, C1009, H1005, LogoB, LogoF,
  TP1001, TP1003 and TP1004; moved C1003, H1004, R1001, TP1002, TP1005,
  TP2001 and U1001; flipped H1012 to the bottom; routed
  encoders/ENC_SW6, Net-(U2002-CH0), Net-(U2002-CH2), Net-(U2002-CH4)
  and 2 more nets; and 17 more changes.
hardware/H4E2/H4E2.kicad_pro: Gergő Törcsvári changed teardrop settings;
  changed 2 ERC rule severities; changed DRC exclusions; changed
  schematic settings.
hardware/H4E2/H4E2.kicad_sch: Gergő Törcsvári removed H1006-H1011;
  changed U1002 wiring; renamed net /encoders/ENC_A2 to
  unconnected-(U3001-GPA3-Pad24); renamed net /encoders/ENC_A3 to
  unconnected-(U3001-GPA5-Pad26); renamed net /encoders/ENC_A7 to
  unconnected-(U3001-GPB3-Pad4); renamed net /encoders/ENC_A8 to
  unconnected-(U3001-GPB0-Pad1); renamed net /encoders/ENC_B2 to
  unconnected-(U3001-GPA4-Pad25); and 5 more changes.
hardware/H4E2/encoder.kicad_sch: Gergő Törcsvári removed C32001-C32003,
  C33001-C33003, C34001-C34003, C35001-C35003, C37001-C37003,
  C38001-C38003 and 18 more; changed D31001 wiring (pin 4 now on
  /encoders/LED_L1_OUT); renamed net /encoders/ENC_A2 to
  unconnected-(U3001-GPA3-Pad24); renamed net /encoders/ENC_A3 to
  unconnected-(U3001-GPA5-Pad26); renamed net /encoders/ENC_A7 to
  unconnected-(U3001-GPB3-Pad4); renamed net /encoders/ENC_A8 to
  unconnected-(U3001-GPB0-Pad1); renamed net /encoders/ENC_B2 to
  unconnected-(U3001-GPA4-Pad25); and 4 more changes.
hardware/H4E2/encoders.kicad_sch: Gergő Törcsvári removed C3002 and
  U3002; changed U3001 wiring (pin 5 now on /encoders/ENC_SW6); renamed
  net /encode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
Parts:
- removed C2004, C2008, C2010, C2013, C23001, C23002, C24001, C24002, C27001, C27002, C28001, C28002, C3002, C32003, C33003, C34003, C35003, C37003, C38003, C39003, C40003: 100nF, Capacitor_SMD:C_0603_1608Metric_Pad1.08x0.95mm_HandSolder
- removed C32001, C32002, C33001, C33002, C34001, C34002, C35001, C35002, C37001, C37002, C38001, C38002, C39001, C39002, C40001, C40002: 1nF, Capacitor_SMD:C_0603_1608Metric_Pad1.08x0.95mm_HandSolder
- removed D23001, D24001, D27001, D28001, D32001, D33001, D34001, D35001, D37001, D38001, D39001, D40001: SK6812MINI-E, LED_SMD:LED_SK6812MINI-E_3.2x2.8mm_P1.5mm_ReverseMount
- removed H1006, H1007, H1008, H1009, H1010, H1011: MountingHole, MountingHole:MountingHole_2.2mm_M2
- removed K23001, K24001, K27001, K28001: ks-20, HALE-git:Gateron_KS-20
- removed LogoB, LogoF: Logo H8E10, HALE-git:Logo H8E10
- removed RN2001, RN2002: 1k, Resistor_SMD:R_Array_Convex_4x0603
- removed SW32001, SW33001, SW34001, SW35001, SW37001, SW38001, SW39001, SW40001: RotaryEncoder_Switch_MP, HALE-git:RotaryEncoder_Alps_EC12E-Switch_Vertical_H20mm
- removed U23001, U24001, U27001, U28001: DRV5055A3xDBZxQ1, Package_TO_SOT_SMD:SOT-23
- removed U3002: MCP23017x-x-SS, Package_SO:SSOP-28_5.3x10.2mm_P0.65mm
- added R2002: 1k, Resistor_SMD:R_0603_1608Metric_Pad0.98x0.95mm_HandSolder, B.Cu at (50.5, 89.0)
- added R2003: 1k, Resistor_SMD:R_0603_1608Metric_Pad0.98x0.95mm_HandSolder, B.Cu at (47.0, 89.0)
- added R2004: 1k, Resistor_SMD:R_0603_1608Metric_Pad0.98x0.95mm_HandSolder, B.Cu at (41.5, 89.0)
- added R2005: 1k, Resistor_SMD:R_0603_1608Metric_Pad0.98x0.95mm_HandSolder, B.Cu at (38.0, 89.0)
- added REF**: Logo H4E2, HALE-git:Logo H4E2, F.Cu at (73.2, 128.5)
- added REF**: Logo H4E2, HALE-git:Logo H4E2, B.Cu at (83.8, 128.5)
- H1005, H1012: moved to B.Cu
- moved C1008 139.8 mm to (87.8, 121.0)
- moved C1009 135.7 mm to (86.2, 105.2), turned to 90 degrees
- moved C3001 78.6 mm to (73.6, 96.7), turned to -90 degrees
- moved TP2001 76.3 mm to (29.4, 92.8)
- moved U3001 74.7 mm to (79.1, 98.9), turned to 0 degrees
- moved TP1002 44.5 mm to (56.5, 86.6)
- moved H1005 40.8 mm to (50.5, 115.8), turned to 180 degrees
- moved C31001 35.3 mm to (102.7, 93.8)
- moved C31002 35.3 mm to (92.7, 93.8)
- moved C31003 35.3 mm to (102.2, 112.5)
- moved D31001 35.3 mm to (97.7, 110.8)
- moved SW31001 35.3 mm to (97.7, 100.3)
- moved C36001 26.4 mm to (92.7, 133.8)
- moved C36002 26.4 mm to (102.7, 133.8)
- moved C36003 26.4 mm to (93.2, 115.1)
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Connections:
- D22001 pad 2: /keys/key2/LED_IN -> /KEYS_LED_DATA_IN
- D26001 pad 2: /keys/key6/LED_IN -> /keys/LED_L1_OUT
- D31001 pad 4: /encoders/encoder1/LED_OUT -> /encoders/LED_L1_OUT
- D36001 pad 2: /encoders/encoder6/LED_IN -> /encoders/LED_L1_OUT
- SW36001 pad S1: /E6_SW -> /encoders/ENC_SW6
- U1002 pad 20: /E6_SW -> unconnected-(U1002-D16-Pad20)
- U2002 pad 2: Net-(RN2001-R2.2) -> /keys/H1
- U2002 pad 4: Net-(RN2001-R4.2) -> /keys/H2
- U2002 pad 6: Net-(RN2002-R2.2) -> /keys/H6
- U2002 pad 8: Net-(RN2002-R4.2) -> /keys/H5
- U3001 pad 1: /encoders/ENC_A8 -> unconnected-(U3001-GPB0-Pad1)
- U3001 pad 2: /encoders/ENC_B8 -> unconnected-(U3001-GPB1-Pad2)
- U3001 pad 23: /encoders/ENC_SW2 -> unconnected-(U3001-GPA2-Pad23)
- U3001 pad 24: /encoders/ENC_A2 -> unconnected-(U3001-GPA3-Pad24)
- U3001 pad 25: /encoders/ENC_B2 -> unconnected-(U3001-GPA4-Pad25)
- U3001 pad 26: /encoders/ENC_A3 -> unconnected-(U3001-GPA5-Pad26)
- U3001 pad 27: /encoders/ENC_B3 -> unconnected-(U3001-GPA6-Pad27)
- U3001 pad 3: /encoders/ENC_SW7 -> unconnected-(U3001-GPB2-Pad3)
- U3001 pad 4: /encoders/ENC_A7 -> unconnected-(U3001-GPB3-Pad4)
- U3001 pad 5: /encoders/ENC_B7 -> /encoders/ENC_SW6
Routing:
- net +5V_LED: track 682.6 -> 312.9 mm, vias 38 -> 15
- net /encoders/I2C_SCL: track 158.4 -> 29.6 mm, vias 3 -> 0
- net +3.3V: track 219.8 -> 92.7 mm, vias 10 -> 6
- net /encoders/RESET: track 144.6 -> 24.2 mm, vias 3 -> 0
- net /E_INT: track 156.7 -> 40.4 mm, vias 3 -> 0
- net /encoders/I2C_SDA: track 147.2 -> 40.1 mm
- net /keys/H4: track 106.8 -> 0.00 mm
- net /keys/H8: track 105.7 -> 0.00 mm
- net +3.3VA: track 265.4 -> 169.4 mm, vias 5 -> 3
- net /keys/H3: track 87.2 -> 0.00 mm
- net /keys/H7: track 85.2 -> 0.00 mm
- net /encoders/ENC_B3: track 74.0 -> 0.00 mm
- net /E6_SW: track 71.2 -> 0.00 mm, vias 2 -> 0
- net /encoders/ENC_B5: track 65.8 -> 0.00 mm
- net /encoders/ENC_B9: track 63.7 -> 0.00 mm
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Other:
- board size 217 x 77.7 mm -> 86 x 77.7 mm
