File: hardware/H4E2/H4E2.kicad_sch (KiCad schematic)
At the start: 34 parts, among them U1001 74AHCT1G125, U1002 XIAO-ESP32-S3-Plus-SMD, U1003 TPS22810DBV, U1004 TPS22810DBV

Commit message: H4E2 "final" design.
hardware/H4E2/H4E2.kicad_pcb: Manufacturing: changed the board outline.
  Gergő Törcsvári: updated from the schematic (added C1008, C1009,
  H1005, R2002-R2005, TP1001, TP1003 and TP1004; removed C2004, C2008,
  C2010, C2013, C3002, C23001 and 47 more; nets changed on 28 pads);
  placed C1008, C1009, C3001, C31001-C31003, C36001-C36003, D31001 and
  10 more; added REF**; removed C1008, C1009, H1005, LogoB, LogoF,
  TP1001, TP1003 and TP1004; moved C1003, H1004, R1001, TP1002, TP1005,
  TP2001 and U1001; flipped H1012 to the bottom; routed
  encoders/ENC_SW6, Net-(U2002-CH0), Net-(U2002-CH2), Net-(U2002-CH4)
  and 2 more nets; and 17 more changes.
hardware/H4E2/H4E2.kicad_pro: Gergő Törcsvári changed teardrop settings;
  changed 2 ERC rule severities; changed DRC exclusions; changed
  schematic settings.
hardware/H4E2/H4E2.kicad_sch: Gergő Törcsvári removed H1006-H1011;
  changed U1002 wiring; renamed net /encoders/ENC_A2 to
  unconnected-(U3001-GPA3-Pad24); renamed net /encoders/ENC_A3 to
  unconnected-(U3001-GPA5-Pad26); renamed net /encoders/ENC_A7 to
  unconnected-(U3001-GPB3-Pad4); renamed net /encoders/ENC_A8 to
  unconnected-(U3001-GPB0-Pad1); renamed net /encoders/ENC_B2 to
  unconnected-(U3001-GPA4-Pad25); and 5 more changes.
hardware/H4E2/encoder.kicad_sch: Gergő Törcsvári removed C32001-C32003,
  C33001-C33003, C34001-C34003, C35001-C35003, C37001-C37003,
  C38001-C38003 and 18 more; changed D31001 wiring (pin 4 now on
  /encoders/LED_L1_OUT); renamed net /encoders/ENC_A2 to
  unconnected-(U3001-GPA3-Pad24); renamed net /encoders/ENC_A3 to
  unconnected-(U3001-GPA5-Pad26); renamed net /encoders/ENC_A7 to
  unconnected-(U3001-GPB3-Pad4); renamed net /encoders/ENC_A8 to
  unconnected-(U3001-GPB0-Pad1); renamed net /encoders/ENC_B2 to
  unconnected-(U3001-GPA4-Pad25); and 4 more changes.
hardware/H4E2/encoders.kicad_sch: Gergő Törcsvári removed C3002 and
  U3002; changed U3001 wiring (pin 5 now on /encoders/ENC_SW6); renamed
  net /encode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
Parts:
- removed H1006, H1007, H1008, H1009, H1010, H1011: MountingHole, MountingHole:MountingHole_2.2mm_M2, symbol Mechanical:MountingHole
Connections:
- net E6_SW: no longer names the net of U1002.20 (D16)
- no-connect marks 14 -> 15
Other:
- sheet encoders ports: added none; removed E6_SW
- title: HALE-H8E10 -> HALE-H4E2
