File: hardware/H4E2/encoders.kicad_sch (KiCad schematic)
At the start: 8 parts, among them U3001 MCP23017x-x-SS, U3002 MCP23017x-x-SS

Commit message: H4E2 "final" design.
hardware/H4E2/H4E2.kicad_pcb: Manufacturing: changed the board outline.
  Gergő Törcsvári: updated from the schematic (added C1008, C1009,
  H1005, R2002-R2005, TP1001, TP1003 and TP1004; removed C2004, C2008,
  C2010, C2013, C3002, C23001 and 47 more; nets changed on 28 pads);
  placed C1008, C1009, C3001, C31001-C31003, C36001-C36003, D31001 and
  10 more; added REF**; removed C1008, C1009, H1005, LogoB, LogoF,
  TP1001, TP1003 and TP1004; moved C1003, H1004, R1001, TP1002, TP1005,
  TP2001 and U1001; flipped H1012 to the bottom; routed
  encoders/ENC_SW6, Net-(U2002-CH0), Net-(U2002-CH2), Net-(U2002-CH4)
  and 2 more nets; and 17 more changes.
hardware/H4E2/H4E2.kicad_pro: Gergő Törcsvári changed teardrop settings;
  changed 2 ERC rule severities; changed DRC exclusions; changed
  schematic settings.
hardware/H4E2/H4E2.kicad_sch: Gergő Törcsvári removed H1006-H1011;
  changed U1002 wiring; renamed net /encoders/ENC_A2 to
  unconnected-(U3001-GPA3-Pad24); renamed net /encoders/ENC_A3 to
  unconnected-(U3001-GPA5-Pad26); renamed net /encoders/ENC_A7 to
  unconnected-(U3001-GPB3-Pad4); renamed net /encoders/ENC_A8 to
  unconnected-(U3001-GPB0-Pad1); renamed net /encoders/ENC_B2 to
  unconnected-(U3001-GPA4-Pad25); and 5 more changes.
hardware/H4E2/encoder.kicad_sch: Gergő Törcsvári removed C32001-C32003,
  C33001-C33003, C34001-C34003, C35001-C35003, C37001-C37003,
  C38001-C38003 and 18 more; changed D31001 wiring (pin 4 now on
  /encoders/LED_L1_OUT); renamed net /encoders/ENC_A2 to
  unconnected-(U3001-GPA3-Pad24); renamed net /encoders/ENC_A3 to
  unconnected-(U3001-GPA5-Pad26); renamed net /encoders/ENC_A7 to
  unconnected-(U3001-GPB3-Pad4); renamed net /encoders/ENC_A8 to
  unconnected-(U3001-GPB0-Pad1); renamed net /encoders/ENC_B2 to
  unconnected-(U3001-GPA4-Pad25); and 4 more changes.
hardware/H4E2/encoders.kicad_sch: Gergő Törcsvári removed C3002 and
  U3002; changed U3001 wiring (pin 5 now on /encoders/ENC_SW6); renamed
  net /encode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
Parts:
- removed C3002: 100nF, Capacitor_SMD:C_0603_1608Metric_Pad1.08x0.95mm_HandSolder, symbol Device:C
- removed U3002: MCP23017x-x-SS, Package_SO:SSOP-28_5.3x10.2mm_P0.65mm, symbol Interface_Expansion:MCP23017x-x-SS
Connections:
- net ENC_A2: no longer names the net of U3001.24 (GPA3)
- net ENC_A3: no longer names the net of U3001.26 (GPA5)
- net ENC_A7: no longer names the net of U3001.4 (GPB3)
- net ENC_A8: no longer names the net of U3001.1 (GPB0)
- net ENC_B2: no longer names the net of U3001.25 (GPA4)
- net ENC_B3: no longer names the net of U3001.27 (GPA6)
- net ENC_B7 renamed ENC_SW6
- net ENC_B8: no longer names the net of U3001.2 (GPB1)
- net ENC_SW2: no longer names the net of U3001.23 (GPA2)
- net ENC_SW7: no longer names the net of U3001.3 (GPB2)
- no-connect marks 6 -> 12
Other:
- removed sheet encoder10
- removed sheet encoder2
- removed sheet encoder3
- removed sheet encoder4
- removed sheet encoder5
- removed sheet encoder7
- removed sheet encoder8
- removed sheet encoder9
