File: hardware/H4E2/keys.kicad_sch (KiCad schematic)
At the start: 23 parts, among them U2001 ME6211C33M5, U2002 MCP3208

Commit message: H4E2 "final" design.
hardware/H4E2/H4E2.kicad_pcb: Manufacturing: changed the board outline.
  Gergő Törcsvári: updated from the schematic (added C1008, C1009,
  H1005, R2002-R2005, TP1001, TP1003 and TP1004; removed C2004, C2008,
  C2010, C2013, C3002, C23001 and 47 more; nets changed on 28 pads);
  placed C1008, C1009, C3001, C31001-C31003, C36001-C36003, D31001 and
  10 more; added REF**; removed C1008, C1009, H1005, LogoB, LogoF,
  TP1001, TP1003 and TP1004; moved C1003, H1004, R1001, TP1002, TP1005,
  TP2001 and U1001; flipped H1012 to the bottom; routed
  encoders/ENC_SW6, Net-(U2002-CH0), Net-(U2002-CH2), Net-(U2002-CH4)
  and 2 more nets; and 17 more changes.
hardware/H4E2/H4E2.kicad_pro: Gergő Törcsvári changed teardrop settings;
  changed 2 ERC rule severities; changed DRC exclusions; changed
  schematic settings.
hardware/H4E2/H4E2.kicad_sch: Gergő Törcsvári removed H1006-H1011;
  changed U1002 wiring; renamed net /encoders/ENC_A2 to
  unconnected-(U3001-GPA3-Pad24); renamed net /encoders/ENC_A3 to
  unconnected-(U3001-GPA5-Pad26); renamed net /encoders/ENC_A7 to
  unconnected-(U3001-GPB3-Pad4); renamed net /encoders/ENC_A8 to
  unconnected-(U3001-GPB0-Pad1); renamed net /encoders/ENC_B2 to
  unconnected-(U3001-GPA4-Pad25); and 5 more changes.
hardware/H4E2/encoder.kicad_sch: Gergő Törcsvári removed C32001-C32003,
  C33001-C33003, C34001-C34003, C35001-C35003, C37001-C37003,
  C38001-C38003 and 18 more; changed D31001 wiring (pin 4 now on
  /encoders/LED_L1_OUT); renamed net /encoders/ENC_A2 to
  unconnected-(U3001-GPA3-Pad24); renamed net /encoders/ENC_A3 to
  unconnected-(U3001-GPA5-Pad26); renamed net /encoders/ENC_A7 to
  unconnected-(U3001-GPB3-Pad4); renamed net /encoders/ENC_A8 to
  unconnected-(U3001-GPB0-Pad1); renamed net /encoders/ENC_B2 to
  unconnected-(U3001-GPA4-Pad25); and 4 more changes.
hardware/H4E2/encoders.kicad_sch: Gergő Törcsvári removed C3002 and
  U3002; changed U3001 wiring (pin 5 now on /encoders/ENC_SW6); renamed
  net /encode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
Parts:
- removed C2004, C2008, C2010, C2013: 100nF, Capacitor_SMD:C_0603_1608Metric_Pad1.08x0.95mm_HandSolder, symbol Device:C
- removed RN2001, RN2002: 1k, Resistor_SMD:R_Array_Convex_4x0603, symbol Device:R_Pack04
- added R2002, R2003, R2004, R2005: 1k, Resistor_SMD:R_0603_1608Metric_Pad0.98x0.95mm_HandSolder, symbol Device:R
Connections:
- net H1: now also U2002.2 (CH1), R2002.1
- net H2: now also U2002.4 (CH3), R2003.2
- net H5: now also U2002.8 (CH7), R2005.2
- net H6: now also U2002.6 (CH5), R2004.2
- net at C2011.2, U2002.7 (CH6): now also R2005.1
- net at C2012.1, U2002.1 (CH0): now also R2002.2
- net at C2007.1, U2002.3 (CH2): now also R2003.1
- net at C2005.2, U2002.5 (CH4): now also R2004.1
Other:
- removed sheet key3
- removed sheet key4
- removed sheet key7
- removed sheet key8
